Commit message: Configurar el plugin hardware interface en el archiu xacro i creació d'un nou launch file per al robot real

File: robot_ws/src/rossy/description/ros2_control.xacro (robot description, xacro)
@@ -1,5 +1,27 @@
 <?xml version="1.0"?>
 <robot xmlns:xacro="http://www.ros.org/wiki/xacro" >
-    <ros2_control name="GazeboSystem" type="system">
+    <ros2_control name="RobotReal" type="system">
+        <hardware>
+            <plugin>rossy_firmware/ArduinoSerialInterface</plugin>
+            <param name="port">/dev/ttyUSB0</param>
+        </hardware>
+        <joint name="joint_roda_esquerra">
+            <command_interface name="velocity">
+                <param name="min">-10</param>
+                <param name="max">10</param>
+            </command_interface>
+            <state_interface name="position" />
+            <state_interface name="velocity" />
+        </joint>
+        <joint name="joint_roda_dreta">
+            <command_interface name="velocity">
+                <param name="min">-10</param>
+                <param name="max">10</param>
+            </command_interface>
+            <state_interface name="velocity" />
+            <state_interface name="position" />
+        </joint>
+    </ros2_control>
+    <!-- <ros2_control name="GazeboSystem" type="system">
         <hardware>
             <plugin>gz_ros2_control/GazeboSimSystem</plugin>
@@ -21,5 +43,5 @@
             <state_interface name="position" />
         </joint>
-    </ros2_control>
+    </ros2_control> -->
     <gazebo>
         <plugin filename="gz_ros2_control-system" name="gz_ros2_control::GazeboSimROS2ControlPlugin">

Commit message: Correcte funcionament robot real i identificació port per l'arduino y el lidar. Falta ajustar característiques del robot per a l'odometría

File: robot_ws/src/rossy/description/ros2_control.xacro (robot description, xacro)
@@ -4,7 +4,7 @@
         <hardware>
             <plugin>rossy_firmware/ArduinoSerialInterface</plugin>
-            <param name="port">/dev/ttyUSB0</param>
+            <param name="port">/dev/arduino</param>
         </hardware>
-        <joint name="joint_roda_esquerra">
+        <joint name="joint_roda_dreta">
             <command_interface name="velocity">
                 <param name="min">-10</param>
@@ -14,5 +14,5 @@
             <state_interface name="velocity" />
         </joint>
-        <joint name="joint_roda_dreta">
+        <joint name="joint_roda_esquerra">
             <command_interface name="velocity">
                 <param name="min">-10</param>
