Commit message: Afegir en el URDF les rodes

File: robot_ws/src/rossy/description/base_robot.xacro (robot description, xacro)
@@ -13,6 +13,8 @@
         <color rgba="0 0 0 1" />
     </material>
+    <!-- LINK BASE -->
     <link name ="link_base">
     </link>
+    <!-- LINK DEL CHASIS -->
     <joint name = "joint_chasis" type ="fixed">
         <parent link ="link_base"/>
@@ -29,3 +31,33 @@
         </visual>
     </link>
+    <!-- LINK RUEDA IZQUIERDA -->
+    <joint name = "joint_roda_esquerra" type = "continuous">
+        <parent link="link_base"/>
+        <child link="roda_esquerra"/>
+        <origin xyz="0 0.175 0" rpy ="-${pi/2} 0 0"/>
+        <axis xyz="0 0 1"/>
+    </joint>
+    <link name = "roda_esquerra">
+        <visual>
+            <geometry>
+                <cylinder radius = "0.05" length="0.04"/>
+            </geometry>
+            <material name = "blue"/>
+        </visual>
+    </link>
+    <!-- LINK RUEDA DERECHA -->
+    <joint name = "joint_roda_dreta" type = "continuous">
+        <parent link="link_base"/>
+        <child link="roda_dreta"/>
+        <origin xyz="0 -0.175 0" rpy ="${pi/2} 0 0"/>
+        <axis xyz="0 0 -1"/>
+    </joint>
+    <link name = "roda_dreta">
+        <visual>
+            <geometry>
+                <cylinder radius = "0.05" length="0.04"/>
+            </geometry>
+            <material name = "blue"/>
+        </visual>
+    </link>
 </robot>

Commit message: Creacio d'una versio de proba URDF del robot, archiu de macros d'inercia y guardat de la configuració de Rviz2

File: robot_ws/src/rossy/description/base_robot.xacro (robot description, xacro)
@@ -1,4 +1,5 @@
 <?xml version="1.0"?>
 <robot xmlns:xacro="http://www.ros.org/wiki/xacro">
+    <xacro:include filename="macros_inercia.xacro"/>
     <material name="white">
         <color rgba="1 1 1 1" />
@@ -30,4 +31,13 @@
             <material name ="white"/>
         </visual>
+        <collision>
+            <origin xyz ="0.15 0 0.075"/>
+            <geometry>
+                <box size ="0.3 0.3 0.15"/>
+            </geometry>
+        </collision>
+        <xacro:inercia_caja masa="1.0" largo="0.3" ancho="0.3" altura="0.15">
+            <origin xyz="0.15 0 0.075" rpy ="0 0 0"/>
+        </xacro:inercia_caja>
     </link>
     <!-- LINK RUEDA IZQUIERDA -->
@@ -45,4 +55,12 @@
             <material name = "blue"/>
         </visual>
+        <collision>
+            <geometry>
+                <cylinder radius = "0.05" length="0.04"/>
+            </geometry>
+        </collision>
+        <xacro:inercia_cilindro masa="0.1" largo="0.04" radio="0.05">
+            <origin xyz="0 0 0" rpy ="0 0 0"/>
+        </xacro:inercia_cilindro>
     </link>
     <!-- LINK RUEDA DERECHA -->
@@ -60,4 +78,34 @@
             <material name = "blue"/>
         </visual>
+        <collision>
+            <geometry>
+                <cylinder radius = "0.05" length="0.04"/>
+            </geometry>
+        </collision>
+        <xacro:inercia_cilindro masa="0.1" largo="0.04" radio="0.05">
+            <origin xyz="0 0 0" rpy ="0 0 0"/>
+        </xacro:inercia_cilindro>
+    </link>
+    <!-- LINK RUEDA MÓVIL -->
+    <joint name="joint_roda_mobil" type="fixed">
+        <parent link="chasis"/>
+        <child link="roda_mobil"/>
+        <origin xyz="0.24 0 0"/>
+    </joint>
+    <link name="roda_mobil">
+        <visual>
+            <geometry>
+                <sphere radius="0.05"/>
+            </geometry>
+            <material name="black"/>
+        </visual>
+        <collision>
+            <geometry>
+                <sphere radius="0.05"/>
+            </geometry>
+        </collision>
+        <xacro:inercia_esfera masa="0.1" radio="0.05">
+            <origin xyz="0 0 0" rpy ="0 0 0"/>
+        </xacro:inercia_esfera>
     </link>
 </robot>

Commit message: Millore varies, creació d'un launch file per Gazebo, un archiu de llançament per aquest i un archiu pont per la nova versió

File: robot_ws/src/rossy/description/base_robot.xacro (robot description, xacro)
@@ -15,9 +15,9 @@
     </material>
     <!-- LINK BASE -->
-    <link name ="link_base">
+    <link name ="base_link">
     </link>
     <!-- LINK DEL CHASIS -->
     <joint name = "joint_chasis" type ="fixed">
-        <parent link ="link_base"/>
+        <parent link ="base_link"/>
         <child link ="chasis"/>
         <origin xyz="-0.1 0 0"/>
@@ -41,7 +41,10 @@
         </xacro:inercia_caja>
     </link>
+    <gazebo reference="chasis">
+        <material>Gazebo/White</material>
+    </gazebo>
     <!-- LINK RUEDA IZQUIERDA -->
     <joint name = "joint_roda_esquerra" type = "continuous">
-        <parent link="link_base"/>
+        <parent link="base_link"/>
         <child link="roda_esquerra"/>
         <origin xyz="0 0.175 0" rpy ="-${pi/2} 0 0"/>
@@ -64,7 +67,10 @@
         </xacro:inercia_cilindro>
     </link>
+    <gazebo reference="roda_esquerra">
+        <material>Gazebo/Blue</material>
+    </gazebo>
     <!-- LINK RUEDA DERECHA -->
     <joint name = "joint_roda_dreta" type = "continuous">
-        <parent link="link_base"/>
+        <parent link="base_link"/>
         <child link="roda_dreta"/>
         <origin xyz="0 -0.175 0" rpy ="${pi/2} 0 0"/>
@@ -87,4 +93,7 @@
         </xacro:inercia_cilindro>
     </link>
+    <gazebo reference="roda_dreta">
+        <material>Gazebo/Blue</material>
+    </gazebo>
     <!-- LINK RUEDA MÓVIL -->
     <joint name="joint_roda_mobil" type="fixed">
@@ -109,3 +118,6 @@
         </xacro:inercia_esfera>
     </link>
+    <gazebo reference="roda_mobil">
+        <material>Gazebo/Black</material>
+    </gazebo>
 </robot>

File: robot_ws/src/rossy/description/robot.urdf.xacro (robot description, xacro)
@@ -2,3 +2,4 @@
 <robot xmlns:xacro="http://www.ros.org/wiki/xacro" name="robot">
     <xacro:include filename = "base_robot.xacro"  />
+    <xacro:include filename = "control_gazebo.xacro"  />
 </robot>

Commit message: Correcció ERROR amb branca git. Tornar a modificar chasis, afegir lidar a gz i correcte funcionamient d'aquest

File: robot_ws/src/rossy/description/base_robot.xacro (robot description, xacro)
@@ -21,9 +21,9 @@
         <parent link ="base_link"/>
         <child link ="chasis"/>
-        <origin xyz="-0.1 0 0"/>
+        <origin xyz="0.1 0 0"/>
     </joint>
     <link name ="chasis">
         <visual>
-            <origin xyz ="0.15 0 0.075"/>
+            <origin xyz ="-0.15 0 0.075"/>
             <geometry>
                 <box size ="0.3 0.3 0.15"/>
@@ -32,5 +32,5 @@
         </visual>
         <collision>
-            <origin xyz ="0.15 0 0.075"/>
+            <origin xyz ="-0.15 0 0.075"/>
             <geometry>
                 <box size ="0.3 0.3 0.15"/>
@@ -38,5 +38,5 @@
         </collision>
         <xacro:inercia_caja masa="1.0" largo="0.3" ancho="0.3" altura="0.15">
-            <origin xyz="0.15 0 0.075" rpy ="0 0 0"/>
+            <origin xyz="-0.15 0 0.075" rpy ="0 0 0"/>
         </xacro:inercia_caja>
     </link>
@@ -100,5 +100,5 @@
         <parent link="chasis"/>
         <child link="roda_mobil"/>
-        <origin xyz="0.24 0 0"/>
+        <origin xyz="-0.24 0 0"/>
     </joint>
     <link name="roda_mobil">

File: robot_ws/src/rossy/description/robot.urdf.xacro (robot description, xacro)
@@ -3,3 +3,4 @@
     <xacro:include filename = "base_robot.xacro"  />
     <xacro:include filename = "control_gazebo.xacro"  />
+    <xacro:include filename = "lidar.xacro"  />
 </robot>

Commit message: Actualització archiu URDF per que sigui igual que el robot real. FALTA CASTER WHEEL

File: robot_ws/src/rossy/description/base_robot.xacro (robot description, xacro)
@@ -2,4 +2,18 @@
 <robot xmlns:xacro="http://www.ros.org/wiki/xacro">
     <xacro:include filename="macros_inercia.xacro"/>
+    <xacro:property name="chassis_length" value="0.250"/>
+    <xacro:property name="chassis_width" value="0.200"/>
+    <xacro:property name="chassis_height" value="0.070"/>
+    <xacro:property name="chassis_mass" value="1.0"/>
+    <xacro:property name="wheel_radius" value="0.033"/>
+    <xacro:property name="wheel_thickness" value="0.026"/>
+    <xacro:property name="wheel_mass" value="0.05"/>
+    <xacro:property name="wheel_offset_x" value="0.0755"/>
+    <xacro:property name="wheel_offset_y" value="0.120"/>
+    <xacro:property name="wheel_offset_z" value="0.004"/>
+    <xacro:property name="caster_wheel_radius" value="0.025"/>
+    <xacro:property name="caster_wheel_mass" value="0.01"/>
+    <xacro:property name="caster_wheel_offset_x" value="0.210"/>
+    <xacro:property name="caster_wheel_offset_z" value="${wheel_offset_z - wheel_radius + caster_wheel_radius}"/>
     <material name="white">
         <color rgba="1 1 1 1" />
@@ -21,26 +35,26 @@
         <parent link ="base_link"/>
         <child link ="chasis"/>
-        <origin xyz="0.1 0 0"/>
+        <origin xyz="${wheel_offset_x} 0 ${wheel_offset_z}"/>
     </joint>
     <link name ="chasis">
         <visual>
-            <origin xyz ="-0.15 0 0.075"/>
+            <origin xyz ="${-chassis_length/2} 0 ${chassis_height/2}"/>
             <geometry>
-                <box size ="0.3 0.3 0.15"/>
+                <box size ="${chassis_length} ${chassis_width} ${chassis_height}"/>
             </geometry>
-            <material name ="white"/>
+            <material name ="black"/>
         </visual>
         <collision>
-            <origin xyz ="-0.15 0 0.075"/>
+            <origin xyz ="${-chassis_length/2} 0 ${chassis_height/2}"/>
             <geometry>
-                <box size ="0.3 0.3 0.15"/>
+                <box size ="${chassis_length} ${chassis_width} ${chassis_height}"/>
             </geometry>
         </collision>
-        <xacro:inercia_caja masa="1.0" largo="0.3" ancho="0.3" altura="0.15">
-            <origin xyz="-0.15 0 0.075" rpy ="0 0 0"/>
+        <xacro:inercia_caja masa="1.0" largo="${chassis_length}" ancho="${chassis_width}" altura="${chassis_height}">
+            <origin xyz="${-chassis_length/2} 0 ${chassis_height/2}" rpy ="0 0 0"/>
         </xacro:inercia_caja>
     </link>
     <gazebo reference="chasis">
-        <material>Gazebo/White</material>
+        <material>Gazebo/Black</material>
     </gazebo>
     <!-- LINK RUEDA IZQUIERDA -->
@@ -48,5 +62,5 @@
         <parent link="base_link"/>
         <child link="roda_esquerra"/>
-        <origin xyz="0 0.175 0" rpy ="-${pi/2} 0 0"/>
+        <origin xyz="0 ${wheel_offset_y} 0" rpy ="-${pi/2} 0 0"/>
         <axis xyz="0 0 1"/>
     </joint>
@@ -54,5 +68,5 @@
         <visual>
             <geometry>
-                <cylinder radius = "0.05" length="0.04"/>
+                <cylinder radius = "${wheel_radius}" length="${wheel_thickness}"/>
             </geometry>
             <material name = "blue"/>
@@ -60,8 +74,8 @@
         <collision>
             <geometry>
-                <cylinder radius = "0.05" length="0.04"/>
+                <cylinder radius = "${wheel_radius}" length="${wheel_thickness}"/>
             </geometry>
         </collision>
-        <xacro:inercia_cilindro masa="0.1" largo="0.04" radio="0.05">
+        <xacro:inercia_cilindro masa="${wheel_mass}" largo="${wheel_thickness}" radio="${wheel_radius}">
             <origin xyz="0 0 0" rpy ="0 0 0"/>
         </xacro:inercia_cilindro>
@@ -74,5 +88,5 @@
         <parent link="base_link"/>
         <child link="roda_dreta"/>
-        <origin xyz="0 -0.175 0" rpy ="${pi/2} 0 0"/>
+        <origin xyz="0 ${-wheel_offset_y} 0" rpy ="${pi/2} 0 0"/>
         <axis xyz="0 0 -1"/>
     </joint>
@@ -80,5 +94,5 @@
         <visual>
             <geometry>
-                <cylinder radius = "0.05" length="0.04"/>
+                <cylinder radius = "${wheel_radius}" length="${wheel_thickness}"/>
             </geometry>
             <material name = "blue"/>
@@ -86,8 +100,8 @@
         <collision>
             <geometry>
-                <cylinder radius = "0.05" length="0.04"/>
+                <cylinder radius = "${wheel_radius}" length="${wheel_thickness}"/>
             </geometry>
         </collision>
-        <xacro:inercia_cilindro masa="0.1" largo="0.04" radio="0.05">
+        <xacro:inercia_cilindro masa="${wheel_mass}" largo="${wheel_thickness}" radio="${wheel_radius}">
             <origin xyz="0 0 0" rpy ="0 0 0"/>
         </xacro:inercia_cilindro>
@@ -100,10 +114,10 @@
         <parent link="chasis"/>
         <child link="roda_mobil"/>
-        <origin xyz="-0.24 0 0"/>
+        <origin xyz="${-caster_wheel_offset_x} 0 ${caster_wheel_offset_z}"/>
     </joint>
     <link name="roda_mobil">
         <visual>
             <geometry>
-                <sphere radius="0.05"/>
+                <sphere radius="${caster_wheel_radius}"/>
             </geometry>
             <material name="black"/>
@@ -111,8 +125,8 @@
         <collision>
             <geometry>
-                <sphere radius="0.05"/>
+                <sphere radius="${caster_wheel_radius}"/>
             </geometry>
         </collision>
-        <xacro:inercia_esfera masa="0.1" radio="0.05">
+        <xacro:inercia_esfera masa="${caster_wheel_mass}" radio="${caster_wheel_radius}">
             <origin xyz="0 0 0" rpy ="0 0 0"/>
         </xacro:inercia_esfera>

File: robot_ws/src/rossy/description/lidar.xacro (robot description, xacro)
@@ -4,10 +4,10 @@
         <parent link="chasis"/>
         <child link="laser_frame"/>
-        <origin xyz="-0.1 0 0.175" rpy="0 0 0"/>
+        <origin xyz="-0.106 0 0.090" rpy="0 0 0"/>
     </joint>
     <link name="laser_frame">
         <visual>
             <geometry>
-                <cylinder radius = "0.05" length="0.04"/>
+                <cylinder radius = "0.035" length="0.03"/>
             </geometry>
             <material name = "black"/>
@@ -15,13 +15,13 @@
         <collision>
             <geometry>
-                <cylinder radius = "0.05" length="0.04"/>
+                <cylinder radius = "0.035" length="0.03"/>
             </geometry>
         </collision>
-        <xacro:inercia_cilindro masa="0.1" largo="0.04" radio="0.05">
+        <xacro:inercia_cilindro masa="0.1" largo="0.03" radio="0.035">
             <origin xyz="0 0 0" rpy ="0 0 0"/>
         </xacro:inercia_cilindro>
     </link>
     <gazebo reference="laser_frame">
-        <material>Gazebo/Black</material>
+        <material>Gazebo/DarkGrey</material>
         <sensor type="gpu_lidar" name="laser">
             <pose> 0 0 0 0 0 0 </pose>

File: robot_ws/src/rossy/description/robot.urdf.xacro (robot description, xacro)
@@ -1,5 +1,5 @@
 <?xml version="1.0"?>
 <robot xmlns:xacro="http://www.ros.org/wiki/xacro" name="robot">
-    <xacro:arg name="usar_ros2_control" default="true"/>
+    <xacro:arg name="use_ros2_control" default="true"/>
     <xacro:include filename = "base_robot.xacro"  />
     <xacro:if value="$(arg use_ros2_control)">

File: robot_ws/src/rossy/description/ros2_control.xacro (robot description, xacro)
@@ -1,5 +1,5 @@
 <?xml version="1.0"?>
 <robot xmlns:xacro="http://www.ros.org/wiki/xacro" >
-    <ros2_control name="RobotReal" type="system">
+    <!-- <ros2_control name="RobotReal" type="system">
         <hardware>
             <plugin>rossy_firmware/ArduinoSerialInterface</plugin>
@@ -22,6 +22,6 @@
             <state_interface name="velocity" />
         </joint>
-    </ros2_control>
-    <!-- <ros2_control name="GazeboSystem" type="system">
+    </ros2_control> -->
+    <ros2_control name="GazeboSystem" type="system">
         <hardware>
             <plugin>gz_ros2_control/GazeboSimSystem</plugin>
@@ -43,5 +43,5 @@
             <state_interface name="position" />
         </joint>
-    </ros2_control> -->
+    </ros2_control>
     <gazebo>
         <plugin filename="gz_ros2_control-system" name="gz_ros2_control::GazeboSimROS2ControlPlugin">

Commit message: S'afegeix l'arxiu YAML per configurar el SLAM del paquet slam_toolbox

File: robot_ws/src/rossy/description/base_robot.xacro (robot description, xacro)
@@ -2,18 +2,18 @@
 <robot xmlns:xacro="http://www.ros.org/wiki/xacro">
     <xacro:include filename="macros_inercia.xacro"/>
-    <xacro:property name="chassis_length" value="0.250"/>
-    <xacro:property name="chassis_width" value="0.200"/>
-    <xacro:property name="chassis_height" value="0.070"/>
-    <xacro:property name="chassis_mass" value="1.0"/>
-    <xacro:property name="wheel_radius" value="0.033"/>
-    <xacro:property name="wheel_thickness" value="0.026"/>
-    <xacro:property name="wheel_mass" value="0.05"/>
-    <xacro:property name="wheel_offset_x" value="0.0755"/>
-    <xacro:property name="wheel_offset_y" value="0.120"/>
-    <xacro:property name="wheel_offset_z" value="0.004"/>
-    <xacro:property name="caster_wheel_radius" value="0.025"/>
-    <xacro:property name="caster_wheel_mass" value="0.01"/>
-    <xacro:property name="caster_wheel_offset_x" value="0.210"/>
-    <xacro:property name="caster_wheel_offset_z" value="${wheel_offset_z - wheel_radius + caster_wheel_radius}"/>
+    <xacro:property name="largo_chassis" value="0.250"/>
+    <xacro:property name="ancho_chassis" value="0.200"/>
+    <xacro:property name="altura_chassis" value="0.070"/>
+    <xacro:property name="masa_chassis" value="1.0"/>
+    <xacro:property name="radio_rueda" value="0.033"/>
+    <xacro:property name="ancho_rueda" value="0.026"/>
+    <xacro:property name="masa_rueda" value="0.05"/>
+    <xacro:property name="rueda_offset_x" value="0.0755"/>
+    <xacro:property name="rueda_offset_y" value="0.120"/>
+    <xacro:property name="rueda_offset_z" value="0.004"/>
+    <xacro:property name="radio_rueda_mobil" value="0.033"/>
+    <xacro:property name="masa_rueda_mobil" value="0.01"/>
+    <xacro:property name="rueda_mobil_offset_x" value="0.210"/>
+    <xacro:property name="rueda_mobil_offset_z" value="-0.004"/>
     <material name="white">
         <color rgba="1 1 1 1" />
@@ -31,26 +31,33 @@
     <link name ="base_link">
     </link>
+    <!-- LINK BASE_FOOTPRINT -->
+    <joint name="base_footprint_joint" type="fixed">
+        <parent link="base_link"/>
+        <child link="base_footprint"/>
+        <origin xyz="0 0 0" rpy="0 0 0"/>
+    </joint>
+    <link name="base_footprint"/>
     <!-- LINK DEL CHASIS -->
     <joint name = "joint_chasis" type ="fixed">
         <parent link ="base_link"/>
         <child link ="chasis"/>
-        <origin xyz="${wheel_offset_x} 0 ${wheel_offset_z}"/>
+        <origin xyz="${rueda_offset_x} 0 ${rueda_offset_z}"/>
     </joint>
     <link name ="chasis">
         <visual>
-            <origin xyz ="${-chassis_length/2} 0 ${chassis_height/2}"/>
+            <origin xyz ="${-largo_chassis/2} 0 ${altura_chassis/2}"/>
             <geometry>
-                <box size ="${chassis_length} ${chassis_width} ${chassis_height}"/>
+                <box size ="${largo_chassis} ${ancho_chassis} ${altura_chassis}"/>
             </geometry>
             <material name ="black"/>
         </visual>
         <collision>
-            <origin xyz ="${-chassis_length/2} 0 ${chassis_height/2}"/>
+            <origin xyz ="${-largo_chassis/2} 0 ${altura_chassis/2}"/>
             <geometry>
-                <box size ="${chassis_length} ${chassis_width} ${chassis_height}"/>
+                <box size ="${largo_chassis} ${ancho_chassis} ${altura_chassis}"/>
             </geometry>
         </collision>
-        <xacro:inercia_caja masa="1.0" largo="${chassis_length}" ancho="${chassis_width}" altura="${chassis_height}">
-            <origin xyz="${-chassis_length/2} 0 ${chassis_height/2}" rpy ="0 0 0"/>
+        <xacro:inercia_caja masa="1.0" largo="${largo_chassis}" ancho="${ancho_chassis}" altura="${altura_chassis}">
+            <origin xyz="${-largo_chassis/2} 0 ${altura_chassis/2}" rpy ="0 0 0"/>
         </xacro:inercia_caja>
     </link>
@@ -62,5 +69,5 @@
         <parent link="base_link"/>
         <child link="roda_esquerra"/>
-        <origin xyz="0 ${wheel_offset_y} 0" rpy ="-${pi/2} 0 0"/>
+        <origin xyz="0 ${rueda_offset_y} 0" rpy ="-${pi/2} 0 0"/>
         <axis xyz="0 0 1"/>
     </joint>
@@ -68,5 +75,5 @@
         <visual>
             <geometry>
-                <cylinder radius = "${wheel_radius}" length="${wheel_thickness}"/>
+                <cylinder radius = "${radio_rueda}" length="${ancho_rueda}"/>
             </geometry>
             <material name = "blue"/>
@@ -74,8 +81,8 @@
         <collision>
             <geometry>
-                <cylinder radius = "${wheel_radius}" length="${wheel_thickness}"/>
+                <cylinder radius = "${radio_rueda}" length="${ancho_rueda}"/>
             </geometry>
         </collision>
-        <xacro:inercia_cilindro masa="${wheel_mass}" largo="${wheel_thickness}" radio="${wheel_radius}">
+        <xacro:inercia_cilindro masa="${masa_rueda}" largo="${ancho_rueda}" radio="${radio_rueda}">
             <origin xyz="0 0 0" rpy ="0 0 0"/>
         </xacro:inercia_cilindro>
@@ -88,5 +95,5 @@
         <parent link="base_link"/>
         <child link="roda_dreta"/>
-        <origin xyz="0 ${-wheel_offset_y} 0" rpy ="${pi/2} 0 0"/>
+        <origin xyz="0 ${-rueda_offset_y} 0" rpy ="${pi/2} 0 0"/>
         <axis xyz="0 0 -1"/>
     </joint>
@@ -94,5 +101,5 @@
         <visual>
             <geometry>
-                <cylinder radius = "${wheel_radius}" length="${wheel_thickness}"/>
+                <cylinder radius = "${radio_rueda}" length="${ancho_rueda}"/>
             </geometry>
             <material name = "blue"/>
@@ -100,8 +107,8 @@
         <collision>
             <geometry>
-                <cylinder radius = "${wheel_radius}" length="${wheel_thickness}"/>
+                <cylinder radius = "${radio_rueda}" length="${ancho_rueda}"/>
             </geometry>
         </collision>
-        <xacro:inercia_cilindro masa="${wheel_mass}" largo="${wheel_thickness}" radio="${wheel_radius}">
+        <xacro:inercia_cilindro masa="${masa_rueda}" largo="${ancho_rueda}" radio="${radio_rueda}">
             <origin xyz="0 0 0" rpy ="0 0 0"/>
         </xacro:inercia_cilindro>
@@ -114,10 +121,10 @@
         <parent link="chasis"/>
         <child link="roda_mobil"/>
-        <origin xyz="${-caster_wheel_offset_x} 0 ${caster_wheel_offset_z}"/>
+        <origin xyz="${-rueda_mobil_offset_x} 0 ${rueda_mobil_offset_z}"/>
     </joint>
     <link name="roda_mobil">
         <visual>
             <geometry>
-                <sphere radius="${caster_wheel_radius}"/>
+                <sphere radius="${radio_rueda_mobil}"/>
             </geometry>
             <material name="black"/>
@@ -125,8 +132,8 @@
         <collision>
             <geometry>
-                <sphere radius="${caster_wheel_radius}"/>
+                <sphere radius="${radio_rueda_mobil}"/>
             </geometry>
         </collision>
-        <xacro:inercia_esfera masa="${caster_wheel_mass}" radio="${caster_wheel_radius}">
+        <xacro:inercia_esfera masa="${masa_rueda_mobil}" radio="${radio_rueda_mobil}">
             <origin xyz="0 0 0" rpy ="0 0 0"/>
         </xacro:inercia_esfera>
